Commit message: change robot color and speed

File: catkin_ws/src/my_robot/urdf/my_robot.xacro (robot description, xacro)
@@ -56,4 +56,7 @@
     </visual>
   </link>
+  <gazebo reference="chassis">
+    <material>Gazebo/FlatBlack</material>
+  </gazebo>
   <link name='right_wheel'>
     <!-- <pose>0 0 0.1 0 0 0</pose> -->
@@ -80,4 +83,7 @@
     </visual>
   </link>
+  <gazebo reference="right_wheel">
+    <material>Gazebo/Yellow</material>
+  </gazebo>
   <joint type="continuous" name="right_wheel_hinge">
     <origin xyz="0 -0.15 0" rpy="0 0 0"/>
@@ -111,4 +117,7 @@
     </visual>
   </link>
+  <gazebo reference="left_wheel">
+    <material>Gazebo/Yellow</material>
+  </gazebo>
   <joint type="continuous" name="left_wheel_hinge">
     <origin xyz="0 0.15 0" rpy="0 0 0"/>
@@ -142,4 +151,7 @@
     </visual>
   </link>
+  <gazebo reference="camera">
+    <material>Gazebo/Grey</material>
+  </gazebo>
   <joint type="continuous" name="camera_joint">
     <origin xyz="0.2 0 0" rpy="0 0 0"/>
