Commit message: basic nav works!

File: project-3-where-am-i/src/my_robot/urdf/my_robot.xacro (robot description, xacro)
@@ -154,5 +154,5 @@
     <material>Gazebo/Grey</material>
   </gazebo>
-  <joint type="continuous" name="camera_joint">
+  <joint type="fixed" name="camera_joint">
     <origin xyz="0.2 0 0" rpy="0 0 0"/>
     <child link="camera"/>
@@ -184,5 +184,5 @@
     </visual>
   </link>
-  <joint type="continuous" name="hokuyo_joint">
+  <joint type="fixed" name="hokuyo_joint">
     <origin xyz="0.15 0 .1" rpy="0 0 0"/>
     <child link="hokuyo"/>
